File: pcb/PicoMemcard-QTPYRP2040BFF/PicoMemcard-qtpyrp2040.kicad_sch (KiCad schematic)
At the start: 9 parts, among them J1 PSX Memory Card Interface, SW1 TS-1187A-B-A-B, SW2 TS-1187A-B-A-B, SW3 TS-1187A-B-A-B, U1 QT_PY_SD_BFF, U2 ADAFRUIT_QT_PY

Commit message: Update led.c
Other:
- title: QT PY RP2040 PicoMemcard -> Adafruit QT Py RP2040 PicoMemcard
Changed lines of the file:
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@@
   (paper "A4")
   (title_block
-    (title "QT PY RP2040 PicoMemcard")
+    (title "Adafruit QT Py RP2040 PicoMemcard")
     (date "2023-08-27")
     (rev "1.0")
     (company "All Around Electronics, LLC.")
+    (comment 1 "Changed RP2040-Zero to Adafruit QT Py RP 2040")
+    (comment 2 "Changed MicroSD SPI to the Adafruit QT Py BFF MicroSD Backpack")
   )
   (junction (at 106.045 146.05) (diameter 0) (color 0 0 0 0)

Commit message: Fix QTPY MicroSD BFF Footprint
Connections:
- net +3.3V: now also U1.5 (3V3); no longer U1.12 (3V3)
- net CS: now also U1.14 (CS); no longer U1.7 (CS)
- net GND: now also U1.6 (GND); no longer U1.13 (GND)
- net MISO: now also U1.3 (MISO); no longer U1.10 (MISO)
- net MOSI: now also U1.4 (MOSI); no longer U1.11 (MOSI)
- net SCK: now also U1.2 (SCK); no longer U1.9 (SCK)
Changed lines of the file:
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@@
     (title "Adafruit QT Py RP2040 PicoMemcard")
     (date "2023-08-31")
-    (rev "1.1")
+    (rev "1.2")
     (company "All Around Electronics, LLC.")
     (comment 1 "Changed RP2040-Zero to Adafruit QT Py RP 2040")
     (comment 2 "Changed MicroSD SPI to the Adafruit QT Py BFF MicroSD Backpack")
     (comment 3 "Connected MicroSD BFF to 3V3 NET (OOF)")
+    (comment 4 "Fixed MicroSD BFF Foorpting ( Mirrored in previous revision )")
   )
   (junction (at 106.045 146.05) (diameter 0) (color 0 0 0 0)
@@
       (effects (font (size 1.27 1.27)) (justify bottom) hide)
     )
-    (pin "12")
-    (pin "13")
-    (pin "10")
-    (pin "11")
-    (pin "7")
-    (pin "9")
-    (instances
-      (project "PicoMemcard-qtpyrp2040"
+    (pin "14")
+    (pin "2")
+    (pin "3")
+    (pin "4")
+    (pin "5")
+    (pin "6")
+    (instances
+      (project "PicoMemcard-qtpyrp2040"
